File: boards/dcesc-ga25/dcesc-ga25.kicad_pcb (KiCad board)
At the start: 2 copper layers, 16 x 10 mm, 11 parts, among them J1 Conn_01x03, J2 Conn_01x03, U1 CH32V003J4M6

Commit message: Розведено.
Parts:
- added C1: 10uF, Capacitor_SMD:C_1206_3216Metric, F.Cu at (185.7, 55.6)
- added C10: 0.1uF, Capacitor_SMD:C_0603_1608Metric, F.Cu at (178.1, 60.3)
- added C11: 100uF, Capacitor_Tantalum_SMD:CP_EIA-3528-12_Kemet-T, F.Cu at (180.3, 80.7)
- added C12: 10uF, Capacitor_SMD:C_0805_2012Metric, F.Cu at (180.3, 84.1)
- added C13: 10uF, Capacitor_SMD:C_0805_2012Metric, F.Cu at (176.9, 80.0)
- added C14: 10uF, Capacitor_SMD:C_1206_3216Metric, F.Cu at (162.6, 60.7)
- added C15: 0.1uF, Capacitor_SMD:C_0603_1608Metric, F.Cu at (160.8, 60.6)
- added C16: 0.1uF, Capacitor_SMD:C_0603_1608Metric, F.Cu at (155.0, 77.9)
- added C17: 0.1uF, Capacitor_SMD:C_0603_1608Metric, F.Cu at (152.8, 87.5)
- added C18: 0.1uF, Capacitor_SMD:C_0603_1608Metric, F.Cu at (166.3, 86.2)
- added C19: 0.1uF, Capacitor_SMD:C_0603_1608Metric, F.Cu at (159.3, 81.2)
- added C20: 0.1uF, Capacitor_SMD:C_0603_1608Metric, F.Cu at (171.9, 73.1)
- added C21: 0.1uF, Capacitor_SMD:C_0603_1608Metric, F.Cu at (160.8, 73.8)
- added C22: 10nF, Capacitor_SMD:C_0603_1608Metric, F.Cu at (161.9, 86.7)
- added C23: 10nF, Capacitor_SMD:C_0603_1608Metric, F.Cu at (160.2, 86.7)
- added C24: 10nF, Capacitor_SMD:C_0603_1608Metric, F.Cu at (158.4, 86.7)
- added C25: 0.1uF, Capacitor_SMD:C_0603_1608Metric, F.Cu at (175.0, 74.4)
- added C27: 0.1uF, Capacitor_SMD:C_0603_1608Metric, F.Cu at (173.6, 77.5)
- added C28: 0.1uF, Capacitor_SMD:C_0603_1608Metric, F.Cu at (149.4, 78.6)
- added C29: 0.1uF, Capacitor_SMD:C_0603_1608Metric, F.Cu at (149.8, 89.6)
- added C3: 0.1uF, Capacitor_SMD:C_0603_1608Metric, F.Cu at (185.9, 57.5)
- added C30: 0.1uF, Capacitor_SMD:C_0603_1608Metric, F.Cu at (149.0, 68.0)
- added C31: 0.1uF, Capacitor_SMD:C_0603_1608Metric, F.Cu at (149.1, 57.2)
- added C32: 0.1uF, Capacitor_SMD:C_0603_1608Metric, F.Cu at (169.3, 86.3)
- added C33: 0.1uF, Capacitor_SMD:C_0603_1608Metric, F.Cu at (117.5, 77.6)
- added C34: 0.1uF, Capacitor_SMD:C_0603_1608Metric, F.Cu at (139.1, 77.6)
- added C35: 0.1uF, Capacitor_SMD:C_0603_1608Metric, F.Cu at (105.7, 72.2)
- added C36: 0.1uF, Capacitor_SMD:C_0603_1608Metric, F.Cu at (127.4, 72.3)
- added C37: 0.1uF, Capacitor_SMD:C_0603_1608Metric, F.Cu at (110.0, 78.6)
- added C38: 0.1uF, Capacitor_SMD:C_0603_1608Metric, F.Cu at (131.4, 78.6)
- added C39: 0.1uF, Capacitor_SMD:C_0603_1608Metric, F.Cu at (113.2, 71.4)
- added C40: 0.1uF, Capacitor_SMD:C_0603_1608Metric, F.Cu at (134.6, 71.4)
- added C41: 33nF, Capacitor_SMD:C_0603_1608Metric, F.Cu at (172.9, 81.7)
- added C42: 33nF, Capacitor_SMD:C_0603_1608Metric, F.Cu at (171.7, 83.2)
- added C43: 33nF, Capacitor_SMD:C_0603_1608Metric, F.Cu at (172.9, 80.2)
- added C44: 33nF, Capacitor_SMD:C_0603_1608Metric, F.Cu at (167.8, 86.2)
- added C45: 10uF, Capacitor_SMD:C_0805_2012Metric, F.Cu at (145.7, 78.6)
- added C46: 10uF, Capacitor_SMD:C_0805_2012Metric, F.Cu at (146.4, 89.4)
- added C47: 10uF, Capacitor_SMD:C_0805_2012Metric, F.Cu at (145.4, 67.9)
- added C48: 10uF, Capacitor_SMD:C_0805_2012Metric, F.Cu at (145.6, 57.2)
- added C49: 1uF, Capacitor_SMD:C_0805_2012Metric, F.Cu at (110.3, 76.8)
- added C5: 0.1uF, Capacitor_SMD:C_0603_1608Metric, F.Cu at (184.8, 67.0)
- added C50: 1uF, Capacitor_SMD:C_0805_2012Metric, F.Cu at (131.8, 76.8)
- added C51: 1uF, Capacitor_SMD:C_0805_2012Metric, F.Cu at (112.8, 73.1)
- added C52: 1uF, Capacitor_SMD:C_0805_2012Metric, F.Cu at (134.1, 73.1)
- added C53: 10uF, Capacitor_SMD:C_1206_3216Metric, F.Cu at (102.0, 77.1)
- added C54: 10uF, Capacitor_SMD:C_1206_3216Metric, F.Cu at (104.4, 77.1)
- added C55: 10uF, Capacitor_SMD:C_1206_3216Metric, F.Cu at (106.8, 77.1)
- added C56: 10uF, Capacitor_SMD:C_1206_3216Metric, F.Cu at (123.6, 77.1)
- added C57: 10uF, Capacitor_SMD:C_1206_3216Metric, F.Cu at (126.0, 77.1)
- added C58: 10uF, Capacitor_SMD:C_1206_3216Metric, F.Cu at (128.4, 77.1)
- added C59: 10uF, Capacitor_SMD:C_1206_3216Metric, F.Cu at (121.2, 72.9)
- added C6: 0.1uF, Capacitor_SMD:C_0603_1608Metric, F.Cu at (182.4, 93.5)
- added C60: 10uF, Capacitor_SMD:C_1206_3216Metric, F.Cu at (118.8, 72.9)
- added C61: 10uF, Capacitor_SMD:C_1206_3216Metric, F.Cu at (116.4, 72.9)
- added C62: 10uF, Capacitor_SMD:C_1206_3216Metric, F.Cu at (142.6, 72.9)
- added C63: 10uF, Capacitor_SMD:C_1206_3216Metric, F.Cu at (140.2, 72.9)
- added C64: 10uF, Capacitor_SMD:C_1206_3216Metric, F.Cu at (137.8, 72.9)
- added C65: 220uF, Capacitor_THT:CP_Radial_D10.0mm_P5.00mm, F.Cu at (196.6, 56.0)
- added C66: 220uF, Capacitor_THT:CP_Radial_D10.0mm_P5.00mm, F.Cu at (196.6, 66.5)
- added C67: 220uF, Capacitor_THT:CP_Radial_D10.0mm_P5.00mm, F.Cu at (196.6, 83.5)
- added C68: 220uF, Capacitor_THT:CP_Radial_D10.0mm_P5.00mm, F.Cu at (196.6, 94.0)
- added C69: 3.3nF, Capacitor_SMD:C_0603_1608Metric, F.Cu at (120.6, 94.0)
- added C7: 82p, Capacitor_SMD:C_0603_1608Metric, F.Cu at (185.7, 68.5)
- added C70: 3.3nF, Capacitor_SMD:C_0603_1608Metric, F.Cu at (142.4, 94.1)
- added C71: 3.3nF, Capacitor_SMD:C_0603_1608Metric, F.Cu at (102.1, 56.0)
- added C72: 3.3nF, Capacitor_SMD:C_0603_1608Metric, F.Cu at (123.9, 56.0)
- added C8: 82p, Capacitor_SMD:C_0603_1608Metric, F.Cu at (185.6, 94.2)
- added C9: 100uF, Capacitor_Tantalum_SMD:CP_EIA-7343-15_Kemet-W, F.Cu at (177.5, 55.1)
- added D1: SMAJ28A, Diode_SMD:D_SMA, F.Cu at (185.6, 52.4)
- added D10: BAT54AW, Package_TO_SOT_SMD:SOT-323_SC-70, F.Cu at (142.7, 77.6)
- added D11: BAT54AW, Package_TO_SOT_SMD:SOT-323_SC-70, F.Cu at (121.2, 52.3)
- added D12: BAT54AW, Package_TO_SOT_SMD:SOT-323_SC-70, F.Cu at (103.6, 72.3)
- added D13: BAT54AW, Package_TO_SOT_SMD:SOT-323_SC-70, F.Cu at (142.6, 52.3)
- added D14: BAT54AW, Package_TO_SOT_SMD:SOT-323_SC-70, F.Cu at (125.3, 72.2)
- added D15: SS24, Diode_SMD:D_SMA, F.Cu at (147.3, 81.3)
- added D16: SS24, Diode_SMD:D_SMA, F.Cu at (147.8, 92.1)
- added D17: SS24, Diode_SMD:D_SMA, F.Cu at (147.6, 70.6)
- added D18: SS24, Diode_SMD:D_SMA, F.Cu at (147.2, 59.9)
- added D19: BAT54AW, Package_TO_SOT_SMD:SOT-323_SC-70, F.Cu at (152.8, 71.3)
- added D2: SS24, Diode_SMD:D_SMA, F.Cu at (181.7, 57.4)
- added D20: LED, LED_SMD:LED_0805_2012Metric, F.Cu at (178.1, 92.4)
- added D3: SS24, Diode_SMD:D_SMA, F.Cu at (183.6, 81.4)
- added D4: BAT54SW, Package_TO_SOT_SMD:SOT-323_SC-70, F.Cu at (163.3, 90.3)
- added D5: BAT54SW, Package_TO_SOT_SMD:SOT-323_SC-70, F.Cu at (159.1, 90.3)
- added D6: BAT54SW, Package_TO_SOT_SMD:SOT-323_SC-70, F.Cu at (152.6, 92.2)
- added D7: BAT54AW, Package_TO_SOT_SMD:SOT-323_SC-70, F.Cu at (102.1, 97.7)
- added D8: BAT54AW, Package_TO_SOT_SMD:SOT-323_SC-70, F.Cu at (119.5, 77.8)
- added D9: BAT54AW, Package_TO_SOT_SMD:SOT-323_SC-70, F.Cu at (123.5, 97.6)
- added FB1: FerriteBead, Inductor_SMD:L_0603_1608Metric, F.Cu at (176.5, 73.7)
- added H1: MountingHole, MountingHole:MountingHole_3.2mm_M3, F.Cu at (106.4, 96.5)
- added H2: MountingHole, MountingHole:MountingHole_3.2mm_M3, F.Cu at (127.9, 96.5)
- added H3: MountingHole, MountingHole:MountingHole_3.2mm_M3, F.Cu at (181.0, 75.0)
- added H4: MountingHole, MountingHole:MountingHole_3.2mm_M3, F.Cu at (116.7, 53.5)
- added H5: MountingHole, MountingHole:MountingHole_3.2mm_M3, F.Cu at (138.2, 53.5)
- added J1: Jumper_2_Open, Jumper:SolderJumper-2_P1.3mm_Open_RoundedPad1.0x1.5mm, B.Cu at (155.7, 67.4)
- added J10: Conn_01x01_Socket, Connector_Wire:SolderWire-2.5sqmm_1x01_D2.4mm_OD4.4mm, F.Cu at (132.5, 53.0)
- added J18: Conn_01x01_Socket, Connector_Wire:SolderWire-6sqmm_1x01_D3.5mm_OD7mm, F.Cu at (196.2, 75.0)
- added J19: Conn_01x01_Socket, Connector_Wire:SolderWire-6sqmm_1x01_D3.5mm_OD7mm, F.Cu at (188.0, 75.0)
- added J3: Conn_01x01_Socket, Connector_Wire:SolderWire-2.5sqmm_1x01_D2.4mm_OD4.4mm, F.Cu at (117.2, 97.0)
- added J4: Conn_01x01_Socket, Connector_Wire:SolderWire-2.5sqmm_1x01_D2.4mm_OD4.4mm, F.Cu at (112.1, 97.0)
- added J5: Conn_01x01_Socket, Connector_Wire:SolderWire-2.5sqmm_1x01_D2.4mm_OD4.4mm, F.Cu at (133.8, 97.0)
- added J6: Conn_01x01_Socket, Connector_Wire:SolderWire-2.5sqmm_1x01_D2.4mm_OD4.4mm, F.Cu at (138.9, 97.0)
- added J7: Conn_01x01_Socket, Connector_Wire:SolderWire-2.5sqmm_1x01_D2.4mm_OD4.4mm, F.Cu at (110.8, 53.0)
- added J8: Conn_01x01_Socket, Connector_Wire:SolderWire-2.5sqmm_1x01_D2.4mm_OD4.4mm, F.Cu at (105.7, 53.0)
- added J9: Conn_01x01_Socket, Connector_Wire:SolderWire-2.5sqmm_1x01_D2.4mm_OD4.4mm, F.Cu at (127.4, 53.0)
- added L1: 10uH, locals:Inductor_NR6028T100M, F.Cu at (179.7, 64.4)
- added L2: 10uH, locals:Inductor_NR6028T100M, F.Cu at (179.2, 88.2)
- added R10: 100k, Resistor_SMD:R_0603_1608Metric, F.Cu at (165.4, 66.1)
- added R11: 100k, Resistor_SMD:R_0603_1608Metric, F.Cu at (175.5, 66.8)
- added R12: 30k, Resistor_SMD:R_0603_1608Metric, F.Cu at (179.3, 69.7)
- added R13: 30k, Resistor_SMD:R_0603_1608Metric, F.Cu at (173.1, 70.3)
- added R14: 0.51R, Resistor_SMD:R_1206_3216Metric, F.Cu at (155.1, 68.3)
- added R15: 1R, Resistor_SMD:R_1206_3216Metric, F.Cu at (162.7, 68.3)
- added R16: 120, Resistor_SMD:R_0603_1608Metric, F.Cu at (155.0, 86.9)
- added R17: 330k, Resistor_SMD:R_0603_1608Metric, F.Cu at (163.4, 86.2)
- added R18: 10k, Resistor_SMD:R_0603_1608Metric, F.Cu at (152.1, 94.8)
- added R19: 10k, Resistor_SMD:R_0603_1608Metric, F.Cu at (148.9, 94.8)
- added R2: 3.3k, Resistor_SMD:R_0603_1608Metric, F.Cu at (188.0, 67.7)
- added R20: 10k, Resistor_SMD:R_0603_1608Metric, F.Cu at (145.8, 94.8)
- added R21: 30k, Resistor_SMD:R_0603_1608Metric, F.Cu at (164.9, 86.2)
- added R22: 100k, Resistor_SMD:R_0603_1608Metric, F.Cu at (161.3, 90.3)
- added R23: 100k, Resistor_SMD:R_0603_1608Metric, F.Cu at (156.9, 90.3)
- added R24: 100k, Resistor_SMD:R_0603_1608Metric, F.Cu at (152.8, 89.7)
- added R25: 100, Resistor_SMD:R_0603_1608Metric, F.Cu at (169.7, 90.3)
- added R26: 100, Resistor_SMD:R_0603_1608Metric, F.Cu at (168.2, 90.3)
- added R27: 100, Resistor_SMD:R_0603_1608Metric, F.Cu at (174.8, 86.6)
- added R28: 100, Resistor_SMD:R_0603_1608Metric, F.Cu at (171.2, 90.3)
- added R29: 100, Resistor_SMD:R_0603_1608Metric, F.Cu at (171.2, 86.6)
- added R30: 100, Resistor_SMD:R_0603_1608Metric, F.Cu at (174.8, 90.3)
- added R31: 100, Resistor_SMD:R_0603_1608Metric, F.Cu at (173.0, 90.3)
- added R32: 100, Resistor_SMD:R_0603_1608Metric, F.Cu at (173.0, 86.6)
- added R33: 100, Resistor_SMD:R_0603_1608Metric, F.Cu at (165.2, 90.3)
- added R34: 100, Resistor_SMD:R_0603_1608Metric, F.Cu at (166.7, 90.3)
- added R35: 330k, Resistor_SMD:R_0603_1608Metric, F.Cu at (176.5, 76.9)
- added R36: 30k, Resistor_SMD:R_0603_1608Metric, F.Cu at (176.5, 78.3)
- added R37: 1k, Resistor_SMD:R_0603_1608Metric, F.Cu at (113.2, 75.0)
- added R38: 1k, Resistor_SMD:R_0603_1608Metric, F.Cu at (134.7, 75.0)
- added R39: 1k, Resistor_SMD:R_0603_1608Metric, F.Cu at (109.5, 74.8)
- added R4: 10k, Resistor_SMD:R_0603_1608Metric, F.Cu at (187.9, 94.9)
- added R40: 1k, Resistor_SMD:R_0603_1608Metric, F.Cu at (131.0, 74.9)
- added R41: 1k, Resistor_SMD:R_0603_1608Metric, F.Cu at (159.4, 84.2)
- added R42: 100k, Resistor_SMD:R_0603_1608Metric, F.Cu at (159.4, 82.8)
- added R43: 10, Resistor_SMD:R_0603_1608Metric, F.Cu at (102.2, 94.2)
- added R44: 10, Resistor_SMD:R_0603_1608Metric, F.Cu at (121.7, 78.0)
- added R45: 10, Resistor_SMD:R_0603_1608Metric, F.Cu at (123.6, 94.5)
- added R46: 10, Resistor_SMD:R_0603_1608Metric, F.Cu at (140.6, 77.6)
- added R47: 10, Resistor_SMD:R_0603_1608Metric, F.Cu at (120.7, 56.0)
- added R48: 10, Resistor_SMD:R_0603_1608Metric, F.Cu at (101.5, 72.2)
- added R49: 10, Resistor_SMD:R_0603_1608Metric, F.Cu at (142.4, 56.0)
- added R5: 3.3k, Resistor_SMD:R_0603_1608Metric, F.Cu at (189.4, 89.0)
- added R50: 10, Resistor_SMD:R_0603_1608Metric, F.Cu at (123.2, 72.2)
- added R51: 3, Resistor_SMD:R_1206_3216Metric, F.Cu at (121.0, 97.0)
- added R52: 3, Resistor_SMD:R_1206_3216Metric, F.Cu at (142.7, 97.0)
- added R53: 3, Resistor_SMD:R_1206_3216Metric, F.Cu at (101.9, 53.0)
- added R54: 3, Resistor_SMD:R_1206_3216Metric, F.Cu at (123.7, 53.0)
- added R55: 5.1k, Resistor_SMD:R_0603_1608Metric, F.Cu at (152.3, 61.0)
- added R56: 5.1k, Resistor_SMD:R_0603_1608Metric, F.Cu at (155.7, 61.9)
- added R57: 3.3k, Resistor_SMD:R_0603_1608Metric, F.Cu at (180.8, 93.5)
- added R57-1: 0.2mOhm, locals:R_SHUNT, B.Cu at (116.8, 82.5)
- added R58-1: 0.2mOhm, locals:R_SHUNT, B.Cu at (106.8, 67.5)
- added R59-1: 0.2mOhm, locals:R_SHUNT, B.Cu at (138.0, 82.5)
- added R6: 100k, Resistor_SMD:R_0603_1608Metric, F.Cu at (187.9, 97.8)
- added R60-1: 0.2mOhm, locals:R_SHUNT, B.Cu at (127.8, 67.5)
- added R61: 5.1k, Resistor_SMD:R_0603_1608Metric, F.Cu at (157.1, 82.3)
- added R62: 5.1k, Resistor_SMD:R_0603_1608Metric, F.Cu at (152.9, 82.4)
- added R63: 100, Resistor_SMD:R_0603_1608Metric, F.Cu at (155.7, 82.4)
- added R64: 100, Resistor_SMD:R_0603_1608Metric, F.Cu at (154.3, 82.4)
- added R7: 30k, Resistor_SMD:R_0603_1608Metric, F.Cu at (170.1, 71.3)
- added R8: 30k, Resistor_SMD:R_0603_1608Metric, F.Cu at (170.5, 67.5)
- added R9: 100k, Resistor_SMD:R_0603_1608Metric, F.Cu at (165.4, 68.1)
- added T1: IPT012N08N5, Package_TO_SOT_SMD:Infineon_PG-HSOF-8-1, F.Cu at (106.2, 86.3)
- added T10: BC847AW, Package_TO_SOT_SMD:SOT-323_SC-70, F.Cu at (168.1, 67.1)
- added T11: IRF5803TRPBF, Package_SO:TSOP-6_1.65x3.05mm_P0.95mm, F.Cu at (173.0, 67.1)
- added T12: AOD4185, Package_TO_SOT_SMD:TO-252-2, F.Cu at (170.3, 61.8)
- added T2: IPT012N08N5, Package_TO_SOT_SMD:Infineon_PG-HSOF-8-1, F.Cu at (116.8, 86.3)
- added T3: IPT012N08N5, Package_TO_SOT_SMD:Infineon_PG-HSOF-8-1, F.Cu at (127.6, 86.3)
- added T4: IPT012N08N5, Package_TO_SOT_SMD:Infineon_PG-HSOF-8-1, F.Cu at (138.2, 86.3)
- added T5: IPT012N08N5, Package_TO_SOT_SMD:Infineon_PG-HSOF-8-1, F.Cu at (117.0, 63.7)
- added T6: IPT012N08N5, Package_TO_SOT_SMD:Infineon_PG-HSOF-8-1, F.Cu at (106.4, 63.7)
- added T7: IPT012N08N5, Package_TO_SOT_SMD:Infineon_PG-HSOF-8-1, F.Cu at (138.4, 63.7)
- added T8: IPT012N08N5, Package_TO_SOT_SMD:Infineon_PG-HSOF-8-1, F.Cu at (127.8, 63.7)
- added T9: BC847AW, Package_TO_SOT_SMD:SOT-323_SC-70, F.Cu at (176.8, 69.6)
- added U10: EG3112, Package_SO:SOP-8_3.9x4.9mm_P1.27mm, F.Cu at (147.9, 85.7)
- added U11: EG3112, Package_SO:SOP-8_3.9x4.9mm_P1.27mm, F.Cu at (147.2, 64.3)
- added U12: EG3112, Package_SO:SOP-8_3.9x4.9mm_P1.27mm, F.Cu at (147.6, 53.5)
- added U13: DRV8870DDA, Package_SO:Texas_HTSOP-8-1EP_3.9x4.9mm_P1.27mm_EP2.95x4.9mm_Mask2.4x3.1mm_ThermalVias, F.Cu at (158.9, 67.0)
- added U14: ATA6561-GAQW-N, Package_SO:SOIC-8_3.9x4.9mm_P1.27mm, F.Cu at (155.0, 82.4)
- added U15: USBLC6-2SC6, Package_TO_SOT_SMD:SOT-23-6, F.Cu at (153.2, 63.9)
- added U2: ST1S14PHR, Package_SO:TI_SO-PowerPAD-8, F.Cu at (185.8, 89.4)
- added U3: MCP1703A-3302, locals:MCP1703, F.Cu at (176.9, 83.0)
- added U4: STM32G431C8Tx, Package_QFP:LQFP-48_7x7mm_P0.5mm, F.Cu at (166.0, 78.1)
- added U5: INA180A4, Package_TO_SOT_SMD:SOT-23-5, F.Cu at (114.7, 77.5)
- added U6: INA180A4, Package_TO_SOT_SMD:SOT-23-5, F.Cu at (136.2, 77.7)
- added U7: INA180A4, Package_TO_SOT_SMD:SOT-23-5, F.Cu at (108.5, 72.3)
- added U8: INA180A4, Package_TO_SOT_SMD:SOT-23-5, F.Cu at (130.2, 72.3)
- added U9: EG3112, Package_SO:SOP-8_3.9x4.9mm_P1.27mm, F.Cu at (147.8, 75.0)
- added X1: Conn_02x02_Top_Bottom, Connector_Molex:Molex_Micro-Fit_3.0_43045-0412_2x02_P3.00mm_Vertical, F.Cu at (167.6, 53.0)
- added X11: Conn_01x03, Connector_JST:JST_ZH_B4B-ZR_1x04_P1.50mm_Vertical, F.Cu at (153.3, 74.7)
- added X12: USB4120-03-C_REVA, locals:GCT_USB4120-03-C_REVA, F.Cu at (154.1, 55.4)
- added X2: Conn_01x03, Connector_JST:JST_XH_B2B-XH-AM_1x02_P2.50mm_Vertical, F.Cu at (160.7, 53.0)
- added X3: Conn_01x03, Connector_JST:JST_ZH_B4B-ZR_1x04_P1.50mm_Vertical, F.Cu at (156.4, 93.5)
- added X4: Conn_01x03, Connector_JST:JST_ZH_B4B-ZR_1x04_P1.50mm_Vertical, F.Cu at (165.2, 93.5)
- added X5: Conn_01x03, Connector_JST:JST_ZH_B4B-ZR_1x04_P1.50mm_Vertical, F.Cu at (169.6, 93.5)
- added X6: Conn_01x03, Connector_JST:JST_ZH_B4B-ZR_1x04_P1.50mm_Vertical, F.Cu at (174.0, 93.5)
- added X7: Conn_01x03, Connector_JST:JST_ZH_B4B-ZR_1x04_P1.50mm_Vertical, F.Cu at (160.8, 93.5)
- added X8: Conn_01x03, Connector_JST:JST_ZH_B3B-ZR_1x03_P1.50mm_Vertical, F.Cu at (182.1, 97.2)
- added X9: Conn_01x03, Connector_JST:JST_ZH_B3B-ZR_1x03_P1.50mm_Vertical, F.Cu at (178.4, 95.0)
- C2: value 0.1uF -> 10uF; footprint Capacitor_SMD:C_0603_1608Metric -> Capacitor_SMD:C_1206_3216Metric
- C26: renamed from C1; value 10uF -> 10nF; footprint Capacitor_SMD:C_0805_2012Metric -> Capacitor_SMD:C_0603_1608Metric
- C4: value 10uF -> 0.1uF; footprint Capacitor_SMD:C_0805_2012Metric -> Capacitor_SMD:C_0603_1608Metric
- J2: value Conn_01x03 -> Jumper_2_Bridged; footprint Connector_JST:JST_PH_S4B-PH-K_1x04_P2.00mm_Horizontal -> Jumper:SolderJumper-2_P1.3mm_Bridged_RoundedPad1.0x1.5mm; moved to B.Cu
- R1: value 4.7k -> 30k
- R3: value 4.7k -> 100k
- TP1: value TestPoint -> BOOT0; footprint TestPoint:TestPoint_Pad_2.0x2.0mm -> TestPoint:TestPoint_Pad_1.0x1.0mm; moved to F.Cu
- U1: value CH32V003J4M6 -> ST1S14PHR; footprint Package_SO:SOP-8_3.9x4.9mm_P1.27mm -> Package_SO:TI_SO-PowerPAD-8
- X10: renamed from J1; footprint Connector_JST:JST_PH_S4B-PH-K_1x04_P2.00mm_Horizontal -> Connector_JST:JST_ZH_B5B-ZR_1x05_P1.50mm_Vertical
- moved FID2 57.1 mm to (197.8, 52.2)
- moved U1 50.2 mm to (186.0, 62.3), turned to 90 degrees
- moved R3 48.2 mm to (187.8, 70.0), turned to 0 degrees
- moved J2 46.5 mm to (162.1, 67.4), turned to 180 degrees
- moved FID1 45.4 mm to (197.8, 97.8)
- moved R1 44.0 mm to (184.7, 70.0), turned to 0 degrees
- moved C26 40.1 mm to (173.5, 74.4), turned to 90 degrees
- moved C2 38.5 mm to (186.9, 81.4)
- moved C4 33.5 mm to (186.6, 84.5), turned to 0 degrees
- moved TP1 31.5 mm to (160.1, 77.8), turned to 0 degrees
- moved X10 16.3 mm to (145.8, 97.3), turned to 0 degrees
Connections:
- C2 pad 1: +5V -> +VM
- C26 pad 1: +5V -> /VDDA
- C4 pad 1: Net-(J2-Pin_1) -> +VM
- J2 pad 1: Net-(J2-Pin_1) -> Net-(J2-A)
- R1 pad 1: Net-(J1-Pin_2) -> +12V
- R1 pad 2: /URX -> Net-(U1-FB)
- R3 pad 1: Net-(J2-Pin_1) -> Net-(U1-FB)
- R3 pad 2: /PWM -> GND
- TP1 pad 1: Net-(U1-PA2) -> /FDCAN1_RX
- U1 pad 1: /URX -> Net-(U1-BOOT)
- U1 pad 2: GND -> unconnected-(U1-PG-Pad2)
- U1 pad 3: Net-(U1-PA2) -> GND
- U1 pad 4: +5V -> Net-(U1-FB)
- U1 pad 5: /PWM -> +VM
- U1 pad 6: /OUT_F -> GND
- U1 pad 7: /OUT_R -> +VM
- U1 pad 8: /SWIO -> /SW1
- X10 pad 1: /SWIO -> GND
- X10 pad 2: Net-(J1-Pin_2) -> Net-(X10-Pin_2)
- X10 pad 3: +5V -> Net-(X10-Pin_3)
- X10 pad 4: GND -> Net-(X10-Pin_4)
Routing:
- net +3.3V: track 0.00 -> 199.8 mm, vias 0 -> 13
- net +12V: track 0.00 -> 183.2 mm, vias 0 -> 6
- net +5V: track 7.58 -> 145.5 mm, vias 0 -> 4
- net +VM: track 0.00 -> 97.0 mm, vias 0 -> 202
- net Net-(U9-HO): track 0.00 -> 70.3 mm, vias 0 -> 2
- net /IC3: track 0.00 -> 69.7 mm, vias 0 -> 2
- net GND: track 0.00 -> 67.9 mm, vias 3 -> 97
- net /IC1: track 0.00 -> 66.8 mm, vias 0 -> 2
- net Net-(U11-LO): track 0.00 -> 66.7 mm, vias 0 -> 2
- net Net-(U12-LO): track 0.00 -> 49.9 mm, vias 0 -> 2
- net /IC4: track 0.00 -> 48.5 mm, vias 0 -> 2
- net /M1.1/OUT: track 0.00 -> 48.3 mm, vias 0 -> 35
- net /IC2: track 0.00 -> 46.5 mm, vias 0 -> 2
- net Net-(U11-HO): track 0.00 -> 45.8 mm, vias 0 -> 2
- net /M4_L: track 0.00 -> 42.0 mm, vias 0 -> 2
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- added copper zone on B.Cu, net +VM
- added copper zone on F.Cu, net +VM
- added copper zone on In1.Cu, net +VM
- added copper zone on In2.Cu, net +VM
- added copper zone on B.Cu, net /M1.1/OUT
- added copper zone on F.Cu, net /M1.1/OUT
- added copper zone on In1.Cu, net /M1.1/OUT
- added copper zone on In2.Cu, net /M1.1/OUT
- added copper zone on F.Cu, net /M1.1/PGND
- added copper zone on B.Cu, net /M1.2/OUT
- added copper zone on F.Cu, net /M1.2/OUT
- added copper zone on In1.Cu, net /M1.2/OUT
- added copper zone on In2.Cu, net /M1.2/OUT
- added copper zone on F.Cu, net /M1.2/PGND
- added copper zone on B.Cu, net /M2.1/OUT
- added copper zone on F.Cu, net /M2.1/OUT
- added copper zone on In1.Cu, net /M2.1/OUT
- added copper zone on In2.Cu, net /M2.1/OUT
- added copper zone on F.Cu, net /M2.1/PGND
- added copper zone on B.Cu, net /M2.2/OUT
- added copper zone on F.Cu, net /M2.2/OUT
- added copper zone on In1.Cu, net /M2.2/OUT
- added copper zone on In2.Cu, net /M2.2/OUT
- added copper zone on F.Cu, net /M2.2/PGND
- added copper zone on F.Cu, net /SW1
- added copper zone on F.Cu, net /SW2
- added copper zone on In1.Cu, net GND
- added copper zone on In2.Cu, net GND
Other:
- board size 16 x 10 mm -> 100 x 50 mm
- copper layers 2 -> 4
- board text added: "0.3A"
- board text added: "0.6A"
- board text added: "DCESC-GA25 v0"
- board text removed: "F"
- board text removed: "G"
- board text removed: "R"
- board text removed: "S"
- board text removed: "T"
- board text removed: "V"

Commit message: Плати замовлено.
Parts:
- moved R57-1 0.30 mm to (116.8, 82.2)
- moved R58-1 0.30 mm to (106.8, 67.8)
- moved R59-1 0.30 mm to (138.0, 82.2)
- moved R60-1 0.30 mm to (127.8, 67.8)
- moved R47 0.12 mm to (120.6, 56.0)
Routing:
- net +VM: vias 202 -> 204
